Commit message: added colors to xacro file

File: src/description/robot_core.xacro (robot description, xacro)
@@ -1,3 +1,15 @@
 <?xml version="1.0"?>
 <robot xmlns:xacro="http://www.ros.org/wiki/xacro">
+<material name="white">
+<color rgba="1 1 1 1" />
+ </material>
+    <material name="orange">
+<color rgba="1 0.3 0.1 1" />
+ </material>
+    <material name="blue">
+<color rgba="0.2 0.2 1 1" />
+ </material>
+    <material name="black">
+<color rgba="0 0 0 1" />
+ </material>
 </robot>

Commit message: base link

File: src/description/robot_core.xacro (robot description, xacro)
@@ -13,3 +13,5 @@
 <color rgba="0 0 0 1" />
  </material>
+<link name="base_link">
+</link>
 </robot>

Commit message: chassis joint

File: src/description/robot_core.xacro (robot description, xacro)
@@ -15,3 +15,8 @@
 <link name="base_link">
 </link>
+<joint name="chassis_joint" type="fixed">
+<parent link="base_link"/>
+<child link="chassis"/>
+<origin xyz="-0.1 0 0"/>
+</joint>
 </robot>

Commit message: CHASSIS AND BASE LINK

File: src/description/robot_core.xacro (robot description, xacro)
@@ -1,22 +1,37 @@
 <?xml version="1.0"?>
 <robot xmlns:xacro="http://www.ros.org/wiki/xacro">
-<material name="white">
-<color rgba="1 1 1 1" />
- </material>
+    <material name="white">
+        <color rgba="1 1 1 1" />
+    </material>
     <material name="orange">
-<color rgba="1 0.3 0.1 1" />
- </material>
+        <color rgba="1 0.3 0.1 1" />
+    </material>
     <material name="blue">
-<color rgba="0.2 0.2 1 1" />
- </material>
+        <color rgba="0.2 0.2 1 1" />
+    </material>
     <material name="black">
-<color rgba="0 0 0 1" />
- </material>
-<link name="base_link">
-</link>
-<joint name="chassis_joint" type="fixed">
-<parent link="base_link"/>
-<child link="chassis"/>
-<origin xyz="-0.1 0 0"/>
-</joint>
+        <color rgba="0 0 0 1" />
+    </material>
+<!-- BASE LINK-->
+    <link name="base_link">
+    </link>
+    <joint name="chassis_joint" type="fixed">
+        <parent link="base_link" />
+        <child link="chassis" />
+        <origin xyz="-0.1 0 0" />
+    </joint>
+<!-- CHASSIS LINK-->
+    <link name="chassis">
+        <visual>
+            <origin xyz="0.15 0 0.075" />
+            <geometry>
+                <box size="0.3 0.3 0.15" />
+            </geometry>
+            <material name=" ">
+                <color rgba=" " />
+            </material>
+            <material name="white" />
+        </visual>
+    </link>
+<!-- LEFT WHEEL LINK-->
 </robot>

Commit message: right wheel

File: src/description/robot_core.xacro (robot description, xacro)
@@ -35,3 +35,18 @@
     </link>
 <!-- LEFT WHEEL LINK-->
+<joint name="left_wheel_joint" type="continous">
+ <parent link="base_link"/>
+<child link="left_wheel"/>
+<origin xyz="0 0.175 0" rpy="-${pi/2} 0 0"/>
+<axis xyz="0 0 1"/>
+</joint>
+<link name="left_wheel">
+        <visual>
+            <origin xyz="0.15 0 0.075" />
+            <geometry>
+                <cylinder radius="0.05" length="0.04"/>
+            </geometry>
+            <material name="blue"/>
+        </visual>
+    </link>
 </robot>

Commit message: caster wheel link

File: src/description/robot_core.xacro (robot description, xacro)
@@ -13,7 +13,8 @@
         <color rgba="0 0 0 1" />
     </material>
-<!-- BASE LINK-->
+    <!-- BASE LINK-->
     <link name="base_link">
     </link>
+    <!-- CHASSIS LINK-->
     <joint name="chassis_joint" type="fixed">
         <parent link="base_link" />
@@ -21,5 +22,4 @@
         <origin xyz="-0.1 0 0" />
     </joint>
-<!-- CHASSIS LINK-->
     <link name="chassis">
         <visual>
@@ -28,24 +28,51 @@
                 <box size="0.3 0.3 0.15" />
             </geometry>
-            <material name=" ">
-                <color rgba=" " />
-            </material>
             <material name="white" />
         </visual>
     </link>
-<!-- LEFT WHEEL LINK-->
-<joint name="left_wheel_joint" type="continous">
- <parent link="base_link"/>
-<child link="left_wheel"/>
-<origin xyz="0 0.175 0" rpy="-${pi/2} 0 0"/>
-<axis xyz="0 0 1"/>
-</joint>
-<link name="left_wheel">
+    <!-- LEFT WHEEL LINK-->
+    <joint name="left_wheel_joint" type="continuous">
+        <parent link="base_link" />
+        <child link="left_wheel" />
+        <origin xyz="0 0.175 0" rpy="-${pi/2} 0 0" />
+        <axis xyz="0 0 1" />
+    </joint>
+    <link name="left_wheel">
         <visual>
             <origin xyz="0.15 0 0.075" />
             <geometry>
-                <cylinder radius="0.05" length="0.04"/>
+                <cylinder radius="0.05" length="0.04" />
             </geometry>
-            <material name="blue"/>
+            <material name="blue" />
+        </visual>
+    </link>
+    <!-- RIGHT WHEEL LINK-->
+    <joint name="right_wheel_joint" type="continuous">
+        <parent link="base_link" />
+        <child link="right_wheel" />
+        <origin xyz="0 -0.175 0" rpy="${pi/2} 0 0" />
+        <axis xyz="0 0 -1" />
+    </joint>
+    <link name="right_wheel">
+        <visual>
+            <origin xyz="0.15 0 0.075" />
+            <geometry>
+                <cylinder radius="0.05" length="0.04" />
+            </geometry>
+            <material name="blue" />
+        </visual>
+    </link>
+    <!-- CASTER WHEEL LINK-->
+    <joint name="caster_wheel_joint" type="fixed">
+        <parent link="chassis" />
+        <child link="caster_wheel" />
+        <origin xyz="0.24 0 0" />
+    </joint>
+    <link>
+        <visual>
+            <geometry>
+            <sphere radius="0.05"/>
+            </geometry>
+            <material name="black"/>
         </visual>
     </link>

Commit message: inertia

File: src/description/robot_core.xacro (robot description, xacro)
@@ -1,4 +1,5 @@
 <?xml version="1.0"?>
 <robot xmlns:xacro="http://www.ros.org/wiki/xacro">
+    <xacro:include filename="inertial_macros.xacro"/>
     <material name="white">
         <color rgba="1 1 1 1" />
@@ -36,4 +37,7 @@
             </geometry>
         </collision>
+ <xacro:inertial_box mass="0.5" x="0.3" y="0.3" z="0.15">
+            <origin xyz="0.15 0 0.75" rpy="0 0 0"/>
+        </xacro:inertial_box>
     </link>
     <!-- LEFT WHEEL LINK-->
@@ -58,4 +62,7 @@
             </geometry>
         </collision>
+        <xacro:inertial_cylinder mass="0.1" length="0.04" radius="0.05">
+            <origin xyz="0 0 0" rpy="0 0 0"/>
+        </xacro:inertial_cylinder>
     </link>
     <!-- RIGHT WHEEL LINK-->
@@ -80,4 +87,7 @@
             </geometry>
         </collision>
+        <xacro:inertial_cylinder mass="0.1" length="0.04" radius="0.05">
+            <origin xyz="0 0 0" rpy="0 0 0"/>
+        </xacro:inertial_cylinder>
     </link>
     <!-- CASTER WHEEL LINK-->
@@ -99,4 +109,7 @@
             </geometry>
         </collision>
+         <xacro:inertial_sphere mass="0.1" radius="0.05">
+            <origin xyz="0 0 0" rpy="0 0 0"/>
+        </xacro:inertial_sphere>
     </link>
 </robot>

Commit message: concept design

File: src/description/robot_core.xacro (robot description, xacro)
@@ -50,5 +50,5 @@
     <link name="left_wheel">
         <visual>
-            <origin xyz="0.15 0 0.075" />
+            <!--origin xyz="0.15 0 0.075" /-->
             <geometry>
                 <cylinder radius="0.05" length="0.04" />
@@ -57,5 +57,5 @@
         </visual>
         <collision>
-            <origin xyz="0.15 0 0.075" />
+            <!-- origin xyz="0.15 0 0.075" /-->
             <geometry>
                 <cylinder radius="0.05" length="0.04" />
@@ -75,5 +75,5 @@
     <link name="right_wheel">
         <visual>
-            <origin xyz="0.15 0 0.075" />
+            <!--origin xyz="0.15 0 0.075" /-->
             <geometry>
                 <cylinder radius="0.05" length="0.04" />
@@ -82,5 +82,5 @@
         </visual>
         <collision>
-            <origin xyz="0.15 0 0.075" />
+            <!--origin xyz="0.15 0 0.075" /-->
             <geometry>
                 <cylinder radius="0.05" length="0.04" />
